File: dddd.kicad_pcb (KiCad board)
At the start: 2 copper layers, 65.5 x 30.9 mm, 25 parts, among them K1 HF32, K2 HF32, K3 HF32, K4 HF32, K5 HF32, Q1 BC817-25_C20069154, Q2 BC817-25_C20069154, Q3 BC817-25_C20069154, Q4 BC817-25_C20069154, Q5 BC817-25_C20069154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

Commit message: Variant Swap: layout2 -> master @ 16:24:34
Parts:
- moved D4 50.4 mm to (147.0, 102.1)
- moved K5 50.4 mm to (150.8, 98.9)
- moved Q5 50.4 mm to (150.6, 105.6)
- moved R5 50.4 mm to (149.6, 102.1)
- moved U5 50.4 mm to (153.3, 83.5)
- moved D2 50.0 mm to (134.4, 102.2)
- moved K2 50.0 mm to (138.3, 98.9)
- moved Q3 50.0 mm to (138.0, 105.7)
- moved R1 50.0 mm to (137.1, 102.2)
- moved U4 50.0 mm to (140.8, 83.6)
- moved D3 30.7 mm to (160.1, 102.1)
- moved K3 30.7 mm to (163.9, 98.9)
- moved Q4 30.7 mm to (163.7, 105.6)
- moved R2 30.7 mm to (162.7, 102.1)
- moved U1 30.7 mm to (166.4, 83.6)
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Routing:
- net GND: track 8.43 -> 0.11 mm
- net Net-(K4-Pad4): track 8.27 -> 4.84 mm
- net Net-(K3-Pad4): track 8.27 -> 4.84 mm
- net Net-(K1-Pad4): track 8.27 -> 4.84 mm
- net Net-(K2-Pad4): track 8.27 -> 4.84 mm
- net Net-(K5-Pad4): track 8.27 -> 4.84 mm
Other:
- board size 65.5 x 30.9 mm -> 65.5 x 61.9 mm
