File: aaaaa.kicad_pcb (KiCad board)
At the start: 2 copper layers, 65.5 x 30.6 mm, 25 parts, among them K1 HF32, K2 HF32, K3 HF32, K4 HF32, K5 HF32, Q1 BC817-25_C20069154, Q2 BC817-25_C20069154, Q3 BC817-25_C20069154, Q4 BC817-25_C20069154, Q5 BC817-25_C20069154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

Commit message: sdcs
Other:
- board text added: "top"
